File: hardware/isc-motorbeep/isc-motorbeep.kicad_pcb (KiCad board)
At the start: 2 copper layers, 0 parts

Commit message: Add placed 4-layer PCB and 3D renders
70 x 50 mm, 4 copper layers, all 69 footprints placed. Not routed: no
tracks, no zones.

Placement is generated by tools/place_board.py, which verifies its own
output -- no courtyard overlaps, nothing off-board, nothing inside the
ESP32 antenna keepout -- and nudges non-anchor passives to the nearest
free spot when a hand-chosen coordinate collides.

Two footprint facts the script encodes, both measured rather than assumed:
pin headers have their origin at pin 1 and extend +Y (J2 reaches 19.6 mm,
so placing it by centre pushes it through the board edge), and U3's
courtyard is inflated to x +-24.3 mm by the antenna keepout, which makes
courtyard-based overlap checks useless next to the module.

The module's antenna overhangs the top edge. L1 is placed directly left
of U2 so SW1/SW2 leave the 0.5 mm-pitch pad column as 4.3 mm straight
runs rather than routing around the package.

3D renders are bare-board: kicad-packages3d is not installed, so no
component bodies.
Parts:
- added BT1: 3x AA, Connector_PinHeader_2.54mm:PinHeader_1x02_P2.54mm_Vertical, F.Cu at (67.0, 43.0)
- added C1: 10uF, Capacitor_SMD:C_0805_2012Metric, F.Cu at (50.5, 38.0)
- added C10: 100nF, Capacitor_SMD:C_0603_1608Metric, F.Cu at (14.0, 25.0)
- added C11: 10uF, Capacitor_SMD:C_0805_2012Metric, F.Cu at (18.0, 25.0)
- added C12: 22uF, Capacitor_SMD:C_0805_2012Metric, F.Cu at (22.0, 25.0)
- added C13: 100nF, Capacitor_SMD:C_0603_1608Metric, F.Cu at (5.00, 9.00)
- added C14: 100nF, Capacitor_SMD:C_0603_1608Metric, F.Cu at (52.0, 13.0)
- added C15: 4.7uF, Capacitor_SMD:C_0805_2012Metric, F.Cu at (52.0, 17.0)
- added C2: 10uF, Capacitor_SMD:C_0805_2012Metric, F.Cu at (50.5, 30.0)
- added C20: 100nF, Capacitor_SMD:C_0603_1608Metric, F.Cu at (13.0, 27.0)
- added C21: 47uF, Capacitor_SMD:C_1210_3225Metric, F.Cu at (24.0, 28.0)
- added C22: 100nF, Capacitor_SMD:C_0603_1608Metric, F.Cu at (13.0, 39.0)
- added C23: 47uF, Capacitor_SMD:C_1210_3225Metric, F.Cu at (24.0, 39.0)
- added C3: 10uF, Capacitor_SMD:C_0805_2012Metric, F.Cu at (54.0, 29.5)
- added C30: 100nF, Capacitor_SMD:C_0603_1608Metric, F.Cu at (32.0, 33.0)
- added C31: 10uF, Capacitor_SMD:C_0805_2012Metric, F.Cu at (36.0, 33.0)
- added C32: 100uF, Capacitor_SMD:C_1210_3225Metric, F.Cu at (40.5, 33.0)
- added C4: 100nF, Capacitor_SMD:C_0603_1608Metric, F.Cu at (58.0, 30.0)
- added C5: 100uF, Capacitor_SMD:C_1210_3225Metric, F.Cu at (61.0, 34.0)
- added D1: MBR0520, Diode_SMD:D_SOD-123, F.Cu at (48.0, 44.0)
- added D2: MBR0520, Diode_SMD:D_SOD-123, F.Cu at (53.0, 46.0)
- added D3: green, LED_SMD:LED_0603_1608Metric, F.Cu at (36.0, 5.00)
- added J1: USB-C, Connector_USB:USB_C_Receptacle_G-Switch_GT-USB-7010ASV, F.Cu at (61.0, 6.00)
- added J2: GPIO header, Connector_PinHeader_2.54mm:PinHeader_1x08_P2.54mm_Vertical, F.Cu at (46.0, 5.00)
- added J3: Stepper 1, Connector_PinHeader_2.54mm:PinHeader_1x04_P2.54mm_Vertical, F.Cu at (3.00, 27.5)
- added J4: Stepper 2, Connector_PinHeader_2.54mm:PinHeader_1x04_P2.54mm_Vertical, F.Cu at (3.00, 39.0)
- added J5: Speaker 4-8R, Connector_PinHeader_2.54mm:PinHeader_1x02_P2.54mm_Vertical, F.Cu at (36.0, 45.0)
- added L1: 2.2uH, Inductor_SMD:L_Bourns-SRN4018, F.Cu at (48.5, 34.0)
- added Q1: BSS138, Package_TO_SOT_SMD:SOT-23, F.Cu at (60.0, 45.0)
- added Q2: MMBT3904, Package_TO_SOT_SMD:SOT-23, F.Cu at (67.0, 19.0)
- added Q3: MMBT3904, Package_TO_SOT_SMD:SOT-23, F.Cu at (67.0, 25.0)
- added R1: 5.1k, Resistor_SMD:R_0603_1608Metric, F.Cu at (52.0, 4.00)
- added R10: 10k, Resistor_SMD:R_0603_1608Metric, F.Cu at (5.00, 5.00)
- added R11: 10k, Resistor_SMD:R_0603_1608Metric, F.Cu at (41.0, 18.0)
- added R12: 1k, Resistor_SMD:R_0603_1608Metric, F.Cu at (40.0, 5.00)
- added R13: 10k, Resistor_SMD:R_0603_1608Metric, F.Cu at (36.0, 18.0)
- added R14: 10k, Resistor_SMD:R_0603_1608Metric, F.Cu at (52.0, 21.0)
- added R15: 10k, Resistor_SMD:R_0603_1608Metric, F.Cu at (67.0, 14.0)
- added R16: 10k, Resistor_SMD:R_0603_1608Metric, F.Cu at (55.0, 27.0)
- added R2: 5.1k, Resistor_SMD:R_0603_1608Metric, F.Cu at (52.0, 8.00)
- added R20: 39k, Resistor_SMD:R_0603_1608Metric, F.Cu at (28.5, 29.0)
- added R21: 10k, Resistor_SMD:R_0603_1608Metric, F.Cu at (28.5, 33.0)
- added R22: 100k, Resistor_SMD:R_0603_1608Metric, F.Cu at (28.5, 37.0)
- added R23: 10k, Resistor_SMD:R_0603_1608Metric, F.Cu at (28.5, 41.0)
- added R24: 10k, Resistor_SMD:R_0603_1608Metric, F.Cu at (28.5, 45.0)
- added R3: 100k, Resistor_SMD:R_0603_1608Metric, F.Cu at (65.0, 33.0)
- added R30: 10k, Resistor_SMD:R_0603_1608Metric, F.Cu at (9.00, 28.0)
- added R31: 100k, Resistor_SMD:R_0603_1608Metric, F.Cu at (9.00, 34.0)
- added R32: 20k, Resistor_SMD:R_0603_1608Metric, F.Cu at (24.0, 31.0)
- added R33: 0.33, Resistor_SMD:R_1206_3216Metric, F.Cu at (18.0, 29.0)
- added R34: 0.33, Resistor_SMD:R_1206_3216Metric, F.Cu at (18.0, 33.0)
- added R4: 68k, Resistor_SMD:R_0603_1608Metric, F.Cu at (64.0, 37.0)
- added R40: 10k, Resistor_SMD:R_0603_1608Metric, F.Cu at (9.00, 40.0)
- added R41: 100k, Resistor_SMD:R_0603_1608Metric, F.Cu at (9.00, 46.0)
- added R42: 20k, Resistor_SMD:R_0603_1608Metric, F.Cu at (24.0, 43.0)
- added R43: 0.33, Resistor_SMD:R_1206_3216Metric, F.Cu at (18.0, 41.0)
- added R44: 0.33, Resistor_SMD:R_1206_3216Metric, F.Cu at (18.0, 45.0)
- added R5: 10R, Resistor_SMD:R_0603_1608Metric, F.Cu at (58.0, 27.0)
- added R50: 100k, Resistor_SMD:R_0603_1608Metric, F.Cu at (41.0, 38.0)
- added SW1: BOOT, Button_Switch_SMD:SW_SPST_SKQG_WithoutStem, F.Cu at (5.00, 22.0)
- added SW2: RESET, Button_Switch_SMD:SW_SPST_SKQG_WithoutStem, F.Cu at (5.00, 15.0)
- added SW3: USER, Button_Switch_SMD:SW_SPST_SKQG_WithoutStem, F.Cu at (38.0, 12.0)
- added U1: USBLC6-2SC6, Package_TO_SOT_SMD:SOT-23-6, F.Cu at (61.0, 14.0)
- added U2: TPS63001, Package_SON:Texas_DRC0010J_ThermalVias, F.Cu at (54.0, 34.0)
- added U3: ESP32-WROOM-32E, RF_Module:ESP32-WROOM-32E, F.Cu at (22.0, 9.00)
- added U4: CP2102N, Package_DFN_QFN:QFN-24-1EP_4x4mm_P0.5mm_EP2.15x2.15mm, F.Cu at (60.0, 22.0)
- added U5: STSPIN220, Package_DFN_QFN:QFN-16-1EP_3x3mm_P0.5mm_EP1.45x1.45mm_ThermalVias, F.Cu at (13.0, 31.0)
- added U6: STSPIN220, Package_DFN_QFN:QFN-16-1EP_3x3mm_P0.5mm_EP1.45x1.45mm_ThermalVias, F.Cu at (13.0, 43.0)
- added U7: MAX98357A, Package_DFN_QFN:QFN-16-1EP_3x3mm_P0.5mm_EP1.45x1.45mm_ThermalVias, F.Cu at (36.0, 38.0)
Other:
- board outline added: 70 x 50 mm
- copper layers 2 -> 4
